Commit message: fix(full-vehicle): synchronize 110-degree zero and 40-110 knee stops

File: model/wheel_leg_v2.0.2/isaac/robot.urdf (robot description, URDF)
Before this commit: robot wheel_leg_v2.0.2_gimbal_fixed_closedchain, 21 links, 20 joints
Joints:
- joint L_joint2: limit lower=-0.08616095279208813 upper=1.0832096460441125 effort=100.0 velocity=100 -> lower=-0.08616095279208813 upper=1.1355695236039427 effort=100.0 velocity=100
- joint R_jonit2: limit lower=-1.0832377220256948 upper=0.08613287681050608 effort=100.0 velocity=100 -> lower=-1.1355975995855245 upper=0.08613287681050608 effort=100.0 velocity=100
